File: pcb/Memory.sch (KiCad schematic (older format))
At the start: 6 parts, among them U7 FM25V05, U8 ST1W008S4ER

Commit message: Clean up Kicad and TCC
Some changes in the
Other:
- note added: "FLASH MEMORY"
- note added: "SD CARD"
- moved on the sheet: R10, R11, R12, R13, U7, U8
