File: pcb/pcb_v1.kicad_pcb (KiCad board)
At the start: 2 copper layers, 95.9 x 90.2 mm, 47 parts, among them IC1 MPU-9250, J1 CONN_01X10, J2 CONN_01X02, U1 ISA_BUS_connector, U2 MSP432P4111, U3 LM317_SOT223, U4 STWD100, U5 ACS711, U6 MCP9701T-E/TTCT-ND, U7 FM25V05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

Commit message: Clean up Kicad and TCC
Some changes in the
Parts:
- added ?: , Connectors:1pin, F.Cu at (140.1, 55.1)
- added ?: , Connectors:1pin, F.Cu at (55.1, 57.6)
- added ?: , Connectors:1pin, F.Cu at (55.1, 131.3)
- added ?: , Connectors:1pin, F.Cu at (140.1, 135.2)
Other:
- outline, holes or cut-outs redrawn
Changed lines of the file:
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@@
     (tracks 830)
     (zones 0)
-    (modules 47)
+    (modules 51)
     (nets 87)
   )
   (page A4)
   (layers
-    (0 F.Cu signal)
-    (31 B.Cu signal)
+    (0 F.Cu signal hide)
+    (31 B.Cu signal hide)
     (32 B.Adhes user hide)
     (33 F.Adhes user hide)
@@
   )
   (setup
-    (last_trace_width 0.25)
+    (last_trace_width 0.2)
     (user_trace_width 0.2)
     (user_trace_width 0.4)
@@
       (padsonsilk false)
       (subtractmaskfromsilk false)
-      (outputformat 1)
+      (outputformat 4)
       (mirror false)
       (drillshape 0)
       (scaleselection 1)
-      (outputdirectory ""))
+      (outputdirectory "layout"))
   )
   (net 0 "")
@@
     (add_net "Net-(R9-Pad2)")
   )
+  (module Connectors:1pin (layer F.Cu)
+    (at 140.09 55.08)
+    (descr "module 1 pin (ou trou mecanique de percage)")
+    (tags DEV)
+    (fp_text reference "" (at 0 -3.048) (layer F.SilkS)
+      (effects (font (size 1 1) (thickness 0.15)))
+    )
+    (fp_text value "" (at 0 3) (layer F.Fab)
+      (effects (font (size 1 1) (thickness 0.15)))
+    )
+    (fp_circle (center 0 0) (end 2 0.8) (layer F.Fab) (width 0.1))
+    (fp_circle (center 0 0) (end 2.6 0) (layer F.CrtYd) (width 0.05))
+    (fp_circle (center 0 0) (end 0 -2.286) (layer F.SilkS) (width 0.12))
+    (pad 1 thru_hole circle (at 0 0) (size 4.064 4.064) (drill 3.048) (layers *.Cu *.Mask))
+  )
+  (module Connectors:1pin (layer F.Cu)
+    (at 55.08 57.62)
+    (descr "module 1 pin (ou trou mecanique de percage)")
+    (tags DEV)
+    (fp_text reference "" (at 0 -3.048) (layer F.SilkS)
+      (effects (font (size 1 1) (thickness 0.15)))
+    )
+    (fp_text value "" (at 0 3) (layer F.Fab)
+      (effects (font (size 1 1) (thickness 0.15)))
+    )
+    (fp_circle (center 0 0) (end 2 0.8) (layer F.Fab) (width 0.1))
+    (fp_circle (center 0 0) (end 2.6 0) (layer F.CrtYd) (width 0.05))
+    (fp_circle (center 0 0) (end 0 -2.286) (layer F.SilkS) (width 0.12))
+    (pad 1 thru_hole circle (at 0 0) (size 4.064 4.064) (drill 3.048) (layers *.Cu *.Mask))
+  )
+  (module Connectors:1pin (layer F.Cu)
+    (at 55.08 131.28)
+    (descr "module 1 pin (ou trou mecanique de percage)")
+    (tags DEV)
+    (fp_text reference "" (at 0 -3.048) (layer F.SilkS)
+      (effects (font (size 1 1) (thickness 0.15)))
+    )
+    (fp_text value "" (at 0 3) (layer F.Fab)
+      (effects (font (size 1 1) (thickness 0.15)))
+    )
+    (fp_circle (center 0 0) (end 2 0.8) (layer F.Fab) (width 0.1))
+    (fp_circle (center 0 0) (end 2.6 0) (layer F.CrtYd) (width 0.05))
+    (fp_circle (center 0 0) (end 0 -2.286) (layer F.SilkS) (width 0.12))
+    (pad 1 thru_hole circle (at 0 0) (size 4.064 4.064) (drill 3.048) (layers *.Cu *.Mask))
+  )
+  (module Connectors:1pin (layer F.Cu)
+    (at 140.09 135.15)
+    (descr "module 1 pin (ou trou mecanique de percage)")
+    (tags DEV)
+    (fp_text reference "" (at 0 -3.048) (layer F.SilkS)
+      (effects (font (size 1 1) (thickness 0.15)))
+    )
+    (fp_text value "" (at 0 3) (layer F.Fab)
+      (effects (font (size 1 1) (thickness 0.15)))
+    )
+    (fp_circle (center 0 0) (end 2 0.8) (layer F.Fab) (width 0.1))
+    (fp_circle (center 0 0) (end 2.6 0) (layer F.CrtYd) (width 0.05))
+    (fp_circle (center 0 0) (end 0 -2.286) (layer F.SilkS) (width 0.12))
+    (pad 1 thru_hole circle (at 0 0) (size 4.064 4.064) (drill 3.048) (layers *.Cu *.Mask))
+  )
   (module Resistors_SMD:R_1206 (layer F.Cu)
     (at 80.264 118.618 45)
@@
     )
   )
+  (gr_arc (start 53 53) (end 53 50) (angle -90) (layer Edge.Cuts) (width 0.15))
+  (gr_arc (start 142.89 53) (end 145.89 53) (angle -90) (layer Edge.Cuts) (width 0.15))
+  (gr_arc (start 142.89 137.17) (end 142.89 140.17) (angle -90) (layer Edge.Cuts) (width 0.15))
+  (gr_arc (start 53 137.17) (end 50 137.17) (angle -90) (layer Edge.Cuts) (width 0.15))
   (gr_line (start 144.526 55.08) (end 138.938 55.08) (layer Dwgs.User) (width 0.15))
   (gr_line (start 138.43 135.15) (end 145.034 135.15) (layer Dwgs.User) (width 0.15))
-  (gr_line (start 140.89 140.17) (end 55 140.17) (layer Edge.Cuts) (width 0.15))
-  (gr_line (start 145.89 135.17) (end 145.89 55) (layer Edge.Cuts) (width 0.15))
-  (gr_arc (start 140.89 135.17) (end 140.89 140.17) (angle -90) (layer Edge.Cuts) (width 0.15))
-  (gr_line (start 140.89 50) (end 55 50) (layer Edge.Cuts) (width 0.15))
-  (gr_arc (start 140.89 55) (end 145.89 55) (angle -90) (layer Edge.Cuts) (width 0.15))
-  (gr_line (start 50 55) (end 50 135.17) (layer Edge.Cuts) (width 0.15))
-  (gr_arc (start 55 55) (end 55 50) (angle -90) (layer Edge.Cuts) (width 0.15))
-  (gr_arc (start 55 135.17) (end 50 135.17) (angle -90) (layer Edge.Cuts) (width 0.15))
+  (gr_line (start 142.89 140.17) (end 53 140.17) (layer Edge.Cuts) (width 0.15))
+  (gr_line (start 145.89 137.17) (end 145.89 53) (layer Edge.Cuts) (width 0.15))
+  (gr_line (start 142.89 50) (end 53 50) (layer Edge.Cuts) (width 0.15))
+  (gr_line (start 50 53) (end 50 137.17) (layer Edge.Cuts) (width 0.15))
   (gr_circle (center 55.08 57.62) (end 58.26 57.62) (layer F.Mask) (width 0.15))
   (gr_line (start 48.9 57.62) (end 59.57 57.62) (angle 90) (layer Dwgs.User) (width 0.15))
