File: pcb/pcb_v1.sch (KiCad schematic (older format))
At the start: 14 parts, among them U1 ISA_BUS_connector, U2 MSP432P4111, Y1 32kHz, Y2 48MHz

Commit message: Clean up Kicad and TCC
Some changes in the
Connections:
- no-connect marks 2 -> 9
Other:
- note added: "CAPACITOR BANK"
- note added: "CURRENT SENSOR"
- note added: "ISA BUS\n"
- note added: "JTAG\n"
- note added: "MEMORY"
- note added: "MPU\n\n"
- note added: "SUPPLY"
- note added: "TEMPERATURE SENSOR"
- note added: "VOLTAGE SENSOR"
- note added: "WATCHDOG\n"
