File: pcb/sensor_inercial.sch (KiCad schematic (older format))
At the start: 4 parts, among them IC1 MPU-9250

Commit message: Clean up Kicad and TCC
Some changes in the
Other:
- moved on the sheet: C14, C15, C16, IC1
Changed lines of the file:
@@
 $Descr A4 11693 8268
 encoding utf-8
-Sheet 8 10
-Title ""
+Sheet 7 10
+Title "Inercial Sensor Schematic"
 Date ""
-Rev ""
-Comp ""
+Rev "1"
+Comp "Universidade de Brasília - Campus Gama"
 Comment1 ""
 Comment2 ""
@@
 L mpu-9250:MPU-9250 IC1
 U 1 1 5B1DB684
-P 5200 3100
-F 0 "IC1" H 4600 4000 50  0000 L CNN
-F 1 "MPU-9250" H 4600 2200 50  0000 L CNN
-F 2 "Housings_DFN_QFN:QFN-24_3x3mm_Pitch0.4mm" H 4600 2100 50  0001 L CNN
-F 3 "https://www.digikey.com/product-detail/en/tdk-invensense/MPU-9250/1428-1019-2-ND/4626449" H 4600 2000 50  0001 L CNN
-F 4 "883-7942" H 4600 1900 50  0001 L CNN "RS"
-F 5 "1428-1019-1-ND" H 4600 1800 50  0001 L CNN "DigiKey"
-	1    5200 3100
+P 6350 4075
+F 0 "IC1" H 5750 4975 50  0000 L CNN
+F 1 "MPU-9250" H 5750 3175 50  0000 L CNN
+F 2 "Housings_DFN_QFN:QFN-24_3x3mm_Pitch0.4mm" H 5750 3075 50  0001 L CNN
+F 3 "https://www.digikey.com/product-detail/en/tdk-invensense/MPU-9250/1428-1019-2-ND/4626449" H 5750 2975 50  0001 L CNN
+F 4 "883-7942" H 5750 2875 50  0001 L CNN "RS"
+F 5 "1428-1019-1-ND" H 5750 2775 50  0001 L CNN "DigiKey"
+	1    6350 4075
 	1    0    0    -1
 $EndComp
 Wire Wire Line
-	4100 2700 4100 2800
-Text HLabel 3550 2250 0    60   Input ~ 0
+	5250 3675 5250 3775
+Text HLabel 4700 3225 0    60   Input ~ 0
 VCC
 $Comp
 L Device:C C14
 U 1 1 5B1DB743
-P 3550 2550
-F 0 "C14" H 3575 2650 50  0000 L CNN
-F 1 "10nF" H 3575 2450 50  0000 L CNN
-F 2 "Capacitors_SMD:C_1206" H 3588 2400 50  0001 C CNN
-F 3 "https://www.digikey.com/product-detail/en/murata-electronics-north-america/GRM033R61E103KA12D/490-7194-2-ND/3900496" H 3550 2550 50  0001 C CNN
-	1    3550 2550
+P 4700 3525
+F 0 "C14" H 4725 3625 50  0000 L CNN
+F 1 "10nF" H 4725 3425 50  0000 L CNN
+F 2 "Capacitors_SMD:C_1206" H 4738 3375 50  0001 C CNN
+F 3 "https://www.digikey.com/product-detail/en/murata-electronics-north-america/GRM033R61E103KA12D/490-7194-2-ND/3900496" H 4700 3525 50  0001 C CNN
+	1    4700 3525
 	1    0    0    -1
 $EndComp
-Connection ~ 4100 2700
+Connection ~ 5250 3675
 Wire Wire Line
-	4500 2500 4100 2500
+	5650 3475 5250 3475
 Wire Wire Line
-	4100 2500 4100 2400
-Connection ~ 4100 2400
+	5250 3475 5250 3375
+Connection ~ 5250 3375
 Wire Wire Line
-	3550 2250 3550 2400
+	4700 3225 4700 3375
 $Comp
 L Device:C C16
 U 1 1 5B1DB835
-P 6450 2950
-F 0 "C16" H 6475 3050 50  0000 L CNN
-F 1 "0.1uF" H 6475 2850 50  0000 L CNN
-F 2 "Capacitors_SMD:C_1206" H 6488 2800 50  0001 C CNN
-F 3 "https://www.digikey.com/product-detail/en/murata-electronics-north-america/GRM033C80J104KE15D/490-10390-1-ND/5026263" H 6450 2950 50  0001 C CNN
-	1    6450 2950
+P 7600 3925
+F 0 "C16" H 7625 4025 50  0000 L CNN
+F 1 "0.1uF" H 7625 3825 50  0000 L CNN
+F 2 "Capacitors_SMD:C_1206" H 7638 3775 50  0001 C CNN
+F 3 "https://www.digikey.com/product-detail/en/murata-electronics-north-america/GRM033C80J104KE15D/490-10390-1-ND/5026263" H 7600 3925 50  0001 C CNN
+	1    7600 3925
 	1    0    0    -1
 $EndComp
 Wire Wire Line
-	5900 2800 6450 2800
+	7050 3775 7600 3775
 $Comp
 L power:GND #PWR014
 U 1 1 5B1DB904
-P 6450 3100
-F 0 "#PWR014" H 6450 2850 50  0001 C CNN
-F 1 "GND" H 6450 2950 50  0000 C CNN
-F 2 "" H 6450 3100 50  0001 C CNN
-F 3 "" H 6450 3100 50  0001 C CNN
-	1    6450 3100
+P 7600 4075
+F 0 "#PWR014" H 7600 3825 50  0001 C CNN
+F 1 "GND" H 7600 3925 50  0000 C CNN
+F 2 "" H 7600 4075 50  0001 C CNN
+F 3 "" H 7600 4075 50  0001 C CNN
+	1    7600 4075
 	1    0    0    -1
 $EndComp
@@
 L Device:C C15
 U 1 1 5B1DB947
-P 3800 2550
-F 0 "C15" H 3825 2650 50  0000 L CNN
-F 1 "0.1uF" H 3825 2450 50  0000 L CNN
-F 2 "Capacitors_SMD:C_1206" H 3838 2400 50  0001 C CNN
-F 3 "https://www.digikey.com/product-detail/en/murata-electronics-north-america/GRM033C80J104KE15D/490-10390-1-ND/5026263" H 3800 2550 50  0001 C CNN
-	1    3800 2550
+P 4950 3525
+F 0 "C15" H 4975 3625 50  0000 L CNN
+F 1 "0.1uF" H 4975 3425 50  0000 L CNN
+F 2 "Capacitors_SMD:C_1206" H 4988 3375 50  0001 C CNN
+F 3 "https://www.digikey.com/product-detail/en/murata-electronics-north-america/GRM033C80J104KE15D/490-10390-1-ND/5026263" H 4950 3525 50  0001 C CNN
+	1    4950 3525
 	1    0    0    -1
 $EndComp
-Connection ~ 3800 2400
+Connection ~ 4950 3375
 Wire Wire Line
-	4500 2800 4400 2800
+	5650 3775 5550 3775
 Wire Wire Line
-	4400 2800 4400 2700
-Connection ~ 4400 2700
-NoConn ~ 5900 3300
-Text HLabel 5925 2500 2    60   Input ~ 0
+	5550 3775 5550 3675
+Connection ~ 5550 3675
+NoConn ~ 7050 4275
+Text HLabel 7075 3475 2    60   Input ~ 0
 SCL/SCLK
-Text HLabel 5925 2600 2    60   Input ~ 0
+Text HLabel 7075 3575 2    60   Input ~ 0
 SDA/SDI
-NoConn ~ 5900 3200
+NoConn ~ 7050 4175
 $Comp
 L power:GND #PWR015
 U 1 1 5B1DB6CC
-P 4100 2800
-F 0 "#PWR015" H 4100 2550 50  0001 C CNN
-F 1 "GND" H 4100 2650 50  0000 C CNN
-F 2 "" H 4100 2800 50  0001 C CNN
-F 3 "" H 4100 2800 50  0001 C CNN
-	1    4100 2800
+P 5250 3775
+F 0 "#PWR015" H 5250 3525 50  0001 C CNN
+F 1 "GND" H 5250 3625 50  0000 C CNN
+F 2 "" H 5250 3775 50  0001 C CNN
+F 3 "" H 5250 3775 50  0001 C CNN
+	1    5250 3775
 	1    0    0    -1
 $EndComp
 Wire Wire Line
-	3550 2700 3800 2700
-Connection ~ 3800 2700
+	4700 3675 4950 3675
+Connection ~ 4950 3675
 Wire Wire Line
-	3550 2400 3800 2400
-Connection ~ 4400 2400
+	4700 3375 4950 3375
+Connection ~ 5550 3375
 $Comp
 L power:GND #PWR016
 U 1 1 5CCE1339
-P 6600 2450
-F 0 "#PWR016" H 6600 2200 50  0001 C CNN
-F 1 "GND" H 6600 2300 50  0000 C CNN
-F 2 "" H 6600 2450 50  0001 C CNN
-F 3 "" H 6600 2450 50  0001 C CNN
-	1    6600 2450
+P 7750 3425
+F 0 "#PWR016" H 7750 3175 50  0001 C CNN
+F 1 "GND" H 7750 3275 50  0000 C CNN
+F 2 "" H 7750 3425 50  0001 C CNN
+F 3 "" H 7750 3425 50  0001 C CNN
+	1    7750 3425
 	1    0    0    -1
 $EndComp
 Wire Wire Line
-	6600 2450 6600 2400
+	7750 3425 7750 3375
 Wire Wire Line
-	6600 2400 5900 2400
-NoConn ~ 5900 2300
-NoConn ~ 5900 2900
-NoConn ~ 5900 3000
+	7750 3375 7050 3375
+NoConn ~ 7050 3275
+NoConn ~ 7050 3875
+NoConn ~ 7050 3975
 Wire Wire Line
-	5925 2500 5900 2500
+	7075 3475 7050 3475
 Wire Wire Line
-	5900 2600 5925 2600
+	7050 3575 7075 3575
 Wire Wire Line
-	4500 2300 4400 2300
+	5650 3275 5550 3275
 Wire Wire Line
-	3800 2300 3800 2400
+	4950 3275 4950 3375
 Wire Wire Line
-	4400 2400 4400 2300
-Connection ~ 4400 2300
+	5550 3375 5550 3275
+Connection ~ 5550 3275
 Wire Wire Line
-	4100 2700 4400 2700
+	5250 3675 5550 3675
 Wire Wire Line
-	4100 2400 4400 2400
+	5250 3375 5550 3375
 Wire Wire Line
-	3800 2400 4100 2400
+	4950 3375 5250 3375
 Wire Wire Line
-	4400 2700 4500 2700
+	5550 3675 5650 3675
 Wire Wire Line
-	3800 2700 4100 2700
+	4950 3675 5250 3675
 Wire Wire Line
-	4400 2400 4500 2400
+	5550 3375 5650 3375
 Wire Wire Line
-	4400 2300 3800 2300
+	5550 3275 4950 3275
+Connection ~ 4700 3375
 $EndSCHEMATC
